File: Board/Autopilot_remote_sender.brd (EAGLE design)
At the start: 27 parts

Commit message: Add schematic Update board
Parts:
- removed D1, D2, D3, D4: 1N4148, diode:SOD110-W
- removed GND: (no value), solpad:SE14
- removed VCC: +, solpad:SE14
- added E$1: (no value), rcl:C0805
- added E$5, E$6: (no value), wirepad:3,17/1,1
Routing:
- net S$28: track 222.0 -> 238.9 mm
- net S$71: track 17.1 -> 7.50 mm
- net S$31: track 111.6 -> 116.6 mm
- net S$73: track 0.00 -> 3.35 mm
- net S$15: track 2.03 -> 4.58 mm
- net S$27: track 213.6 -> 211.1 mm
- net S$72: track 12.8 -> 15.0 mm
- net S$13: track 2.03 -> 0.00 mm
- net S$30: track 84.1 -> 82.2 mm
- net S$29: track 174.7 -> 175.3 mm
Other:
- board text added: "_"
- board text removed: "-"

Commit message: Add gerber files
Parts:
- removed E$17, E$18, E$22, E$23, E$24, E$25: (no value), holes:2,8-PAD
Other:
- board outline added: 62 x 128.5 mm
